File: ECAD/pocket_sprite.kicad_pcb (KiCad board)
At the start: 2 copper layers, 125 x 46 mm, 18 parts, among them J1 Screw_Terminal_01x02, Q1 AO3400A, SW1 DS04-254-2-01BK-SMT, SW3 BUTTON, U1 1.8_TFT_LCD_Display_Module, U2 ESP32-S3

Commit message: redid gerbers
Parts:
- moved J1 10.1 mm to (164.9, 65.7), turned to -90 degrees
- moved PAD1 5.13 mm to (155.0, 66.6)
Routing:
- net XIAO_BAT+: track 11.2 -> 10.4 mm
- net GND: vias 47 -> 49
